Commit message: added: - lidar camera fusion package:   - body preprocess node for removing bed plane   - manual segmentation window - massage path tool package - sharing guide   fix: - stitched image result accurate - urdf rotation, offset and webcam calibration value

File: src/lidar_camera_fusion/urdf/scanner_bridge.urdf (robot description, URDF)
Before this commit: robot medical_scanner, 5 links, 4 joints
Joints:
- joint camera_to_optical: origin xyz=0 0.06 0 rpy=-1.5708 0 -1.5708 -> xyz=0.035 0.06 0.0 rpy=0 0 0
- joint gantry_to_camera: origin xyz=0.07 0.0 -0.03 rpy=0 1.5708 3.14159 -> xyz=0.07 0.0 -0.03 rpy=3.14159 0 1.5708
