Commit message: Update gantry position topic massage type and update massage tool

File: src/lidar_camera_fusion/urdf/scanner_bridge.urdf (robot description, URDF)
Before this commit: robot medical_scanner, 5 links, 4 joints
Links:
- link base_link: geometry collision box size=0.3 0.3 0.1; visual box size=2.08 1.0 0.04
- link camera_link: geometry collision box size=0.08 0.08 0.08; visual box size=0.1 0.025 0.024
- link lidar_link: geometry collision cylinder length=0.06 radius=0.04; visual cylinder length=0.025 radius=0.069
Joints:
- joint camera_to_optical: origin xyz=0.035 0.06 0.0 rpy=0 0 0 -> xyz=0.035 0.04 0.0 rpy=0 0 0
- joint gantry_joint: origin xyz=0 0 0.72 rpy=0 0 0 -> xyz=0 0 0.888 rpy=0 0 0
- joint gantry_to_camera: origin xyz=0.07 0.0 -0.03 rpy=3.14159 0 1.5708 -> xyz=0.043 0.0 -0.0615 rpy=3.14159 0 1.5708
